File: kicad/pico-wiegand/pico-wiegand.kicad_sch (KiCad schematic)
At the start: 23 parts, among them J1 Power/GND, J2 Reader, J3 Door Contact, J4 Push Button, J5 Lock Relay, Q1 BSS138, Q2 BSS138, Q3 BSS138, Q4 BSS138, U1 Pico

Commit message: Updated schematics with HID LED
Parts:
- K1: value (none) -> SPDT
- R8: value 220 -> (none)
Connections:
- net DOOR: now also U1.19 (GPIO14); no longer U1.21 (GPIO16)
- net LED: now also U1.20 (GPIO15); no longer U1.22 (GPIO17)
- net CLOCK renamed D0
- net D0: no longer Q1.2 (S), R1.2, U1.25 (GPIO19)
- net DATA renamed D1
- net D1: now also U1.21 (GPIO16); no longer U1.24 (GPIO18)
- new net: Q1.2 (S), R1.2, U1.22 (GPIO17)
Other:
- moved on the sheet: R8, U1
